Commit message: updated teleop
updated teleop

File: Project4_SLAM/my_robot/urdf/my_robot.xacro (robot description, xacro)
@@ -141,5 +141,5 @@
   <!-- left_wheeljoints -->
   <joint type="continuous" name="left_wheel_hinge">
-    <origin xyz="0 0.125 0" rpy="0 0 0"/>
+    <origin xyz="0 0.15 0" rpy="0 0 0"/>
     <child link="left_wheel"/>
     <parent link="chassis"/>
@@ -150,5 +150,5 @@
   <!-- right_wheeljoints -->
   <joint type="continuous" name="right_wheel_hinge">
-    <origin xyz="0 -0.125 0" rpy="0 0 0"/>
+    <origin xyz="0 -0.15 0" rpy="0 0 0"/>
     <child link="right_wheel"/>
     <parent link="chassis"/>
